File: ShowMeShield.brd (EAGLE design)
At the start: 84.3 x 50 mm, 70 parts, among them Q0 MOSFET-N-044020001, Q1 MOSFET-N-044020001, Q10 MOSFET-N-044020001, Q11 MOSFET-N-044020001, Q12 MOSFET-N-044020001, Q13 MOSFET-N-044020001, Q14 MOSFET-N-044020001, Q15 MOSFET-N-044020001, Q16 MOSFET-N-044020001, Q17 MOSFET-N-044020001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

Commit message: 1.5
Parts:
- ARDUINO: value ARDUINO_SHIELD_SFNO_SILK -> ARDUINO_SHIELDNO_SILK; device MCP:DUEMILANOVE_VIAS -> SPCoast:DUEMILANOVE_VIAS
- moved U$1 2.54 mm to (4.62, 5.51)
- moved ARDUINO 0.13 mm to (16.3, 1.27)
Routing:
- net VCC: track 200.6 -> 199.0 mm
- added copper zone on layer 1, net VCC
Other:
- outline, holes or cut-outs redrawn
- board text added: "2014.07"
- board text added: "3.3"
- board text added: "5v"
- board text added: "Gnd"
- board text added: "RESET"
- board text added: "SPCoast"
- board text added: "V1.5"
- board text added: "Vin"
- board text removed: "V1.4"
