File: ShowMeShield.sch (EAGLE design)
At the start: 70 parts, among them Q0 MOSFET-N-044020001, Q1 MOSFET-N-044020001, Q10 MOSFET-N-044020001, Q11 MOSFET-N-044020001, Q12 MOSFET-N-044020001, Q13 MOSFET-N-044020001, Q14 MOSFET-N-044020001, Q15 MOSFET-N-044020001, Q16 MOSFET-N-044020001, Q17 MOSFET-N-044020001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

Commit message: 1.5
Parts:
- ARDUINO: value ARDUINO_SHIELD_SFNO_SILK -> ARDUINO_SHIELDNO_SILK; device MCP:ARDUINO_SHIELD_SFNO_SILK -> SPCoast:ARDUINO_SHIELDNO_SILK
Changed lines of the file:
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@@
 <?xml version="1.0" encoding="utf-8"?>
 <!DOCTYPE eagle SYSTEM "eagle.dtd">
-<eagle version="6.4">
+<eagle version="6.6.0">
 <drawing>
 <settings>
@@
 <part name="P+3" library="supply1" deviceset="V+" device=""/>
 <part name="P+6" library="supply1" deviceset="V+" device=""/>
-<part name="ARDUINO" library="MCP" deviceset="ARDUINO_SHIELD_SF" device="NO_SILK"/>
+<part name="ARDUINO" library="SPCoast" deviceset="ARDUINO_SHIELD" device="NO_SILK" value="ARDUINO_SHIELDNO_SILK"/>
 <part name="GND5" library="SparkFun" deviceset="GND" device=""/>
 <part name="GND1" library="SparkFun" deviceset="GND" device=""/>
@@
 <instance part="P+3" gate="1" x="200.66" y="139.7"/>
 <instance part="P+6" gate="1" x="40.64" y="35.56"/>
-<instance part="ARDUINO" gate="G$1" x="66.04" y="35.56"/>
+<instance part="ARDUINO" gate="SHIELD" x="66.04" y="35.56"/>
 <instance part="GND5" gate="1" x="53.34" y="7.62"/>
 <instance part="GND1" gate="1" x="35.56" y="127"/>
@@
 <wire x1="53.34" y1="30.48" x2="38.1" y2="30.48" width="0.1524" layer="91"/>
 <pinref part="P+4" gate="VCC" pin="VCC"/>
-<pinref part="ARDUINO" gate="G$1" pin="5V"/>
+<pinref part="ARDUINO" gate="SHIELD" pin="5V"/>
 </segment>
 <segment>
@@
 <wire x1="78.74" y1="53.34" x2="81.28" y2="53.34" width="0.1524" layer="91"/>
 <label x="81.28" y="53.34" size="1.27" layer="95" xref="yes"/>
-<pinref part="ARDUINO" gate="G$1" pin="RX"/>
+<pinref part="ARDUINO" gate="SHIELD" pin="RX"/>
 </segment>
 </net>
@@
 <wire x1="78.74" y1="50.8" x2="81.28" y2="50.8" width="0.1524" layer="91"/>
 <label x="81.28" y="50.8" size="1.27" layer="95" xref="yes"/>
-<pinref part="ARDUINO" gate="G$1" pin="TX"/>
+<pinref part="ARDUINO" gate="SHIELD" pin="TX"/>
 </segment>
 </net>
@@
 <wire x1="78.74" y1="45.72" x2="81.28" y2="45.72" width="0.1524" layer="91"/>
 <label x="81.28" y="45.72" size="1.27" layer="95" xref="yes"/>
-<pinref part="ARDUINO" gate="G$1" pin="D2"/>
+<pinref part="ARDUINO" gate="SHIELD" pin="D2"/>
 </segment>
 </net>
@@
 <wire x1="78.74" y1="43.18" x2="81.28" y2="43.18" width="0.1524" layer="91"/>
 <label x="81.28" y="43.18" size="1.27" layer="95" xref="yes"/>
-<pinref part="ARDUINO" gate="G$1" pin="*D3"/>
+<pinref part="ARDUINO" gate="SHIELD" pin="*D3"/>
 </segment>
 </net>
@@
 <wire x1="78.74" y1="40.64" x2="81.28" y2="40.64" width="0.1524" layer="91"/>
 <label x="81.28" y="40.64" size="1.27" layer="95" xref="yes"/>
-<pinref part="ARDUINO" gate="G$1" pin="D4"/>
+<pinref part="ARDUINO" gate="SHIELD" pin="D4"/>
 </segment>
 </net>
@@
 <wire x1="78.74" y1="38.1" x2="81.28" y2="38.1" width="0.1524" layer="91"/>
 <label x="81.28" y="38.1" size="1.27" layer="95" xref="yes"/>
-<pinref part="ARDUINO" gate="G$1" pin="*D5"/>
+<pinref part="ARDUINO" gate="SHIELD" pin="*D5"/>
 </segment>
 </net>
@@
 <wire x1="78.74" y1="35.56" x2="81.28" y2="35.56" width="0.1524" layer="91"/>
 <label x="81.28" y="35.56" size="1.27" layer="95" xref="yes"/>
-<pinref part="ARDUINO" gate="G$1" pin="*D6"/>
+<pinref part="ARDUINO" gate="SHIELD" pin="*D6"/>
 </segment>
 </net>
@@
 <wire x1="78.74" y1="25.4" x2="81.28" y2="25.4" width="0.1524" layer="91"/>
 <label x="81.28" y="25.4" size="1.27" layer="95" xref="yes"/>
-<pinref part="ARDUINO" gate="G$1" pin="*D10"/>
+<pinref part="ARDUINO" gate="SHIELD" pin="*D10"/>
 </segment>
 <segment>
@@
 <wire x1="53.34" y1="53.34" x2="50.8" y2="53.34" width="0.1524" layer="91"/>
 <label x="50.8" y="53.34" size="1.27" layer="95" rot="R180" xref="yes"/>
-<pinref part="ARDUINO" gate="G$1" pin="A0"/>
+<pinref part="ARDUINO" gate="SHIELD" pin="A0"/>
 </segment>
 <segment>
@@
 <wire x1="53.34" y1="50.8" x2="50.8" y2="50.8" width="0.1524" layer="91"/>
 <label x="50.8" y="50.8" size="1.27" layer="95" rot="R180" xref="yes"/>
-<pinref part="ARDUINO" gate="G$1" pin="A1"/>
+<pinref part="ARDUINO" gate="SHIELD" pin="A1"/>
 </segment>
 <segment>
@@
 <wire x1="53.34" y1="48.26" x2="50.8" y2="48.26" width="0.1524" layer="91"/>
 <label x="50.8" y="48.26" size="1.27" layer="95" rot="R180" xref="yes"/>
-<pinref part="ARDUINO" gate="G$1" pin="A2"/>
+<pinref part="ARDUINO" gate="SHIELD" pin="A2"/>
 </segment>
 <segment>
@@
 <wire x1="53.34" y1="45.72" x2="50.8" y2="45.72" width="0.1524" layer="91"/>
 <label x="50.8" y="45.72" size="1.27" layer="95" rot="R180" xref="yes"/>
-<pinref part="ARDUINO" gate="G$1" pin="A3"/>
+<pinref part="ARDUINO" gate="SHIELD" pin="A3"/>
 </segment>
 <segment>
@@
 <wire x1="53.34" y1="43.18" x2="50.8" y2="43.18" width="0.1524" layer="91"/>
 <label x="50.8" y="43.18" size="1.27" layer="95" rot="R180" xref="yes"/>
-<pinref part="ARDUINO" gate="G$1" pin="A4"/>
+<pinref part="ARDUINO" gate="SHIELD" pin="A4"/>
 </segment>
 <segment>
@@
 <wire x1="53.34" y1="40.64" x2="50.8" y2="40.64" width="0.1524" layer="91"/>
 <label x="50.8" y="40.64" size="1.27" layer="95" rot="R180" xref="yes"/>
-<pinref part="ARDUINO" gate="G$1" pin="A5"/>
+<pinref part="ARDUINO" gate="SHIELD" pin="A5"/>
 </segment>
 <segment>
@@
 <wire x1="78.74" y1="33.02" x2="81.28" y2="33.02" width="0.1524" layer="91"/>
 <label x="81.28" y="33.02" size="1.27" layer="95" xref="yes"/>
-<pinref part="ARDUINO" gate="G$1" pin="D7"/>
+<pinref part="ARDUINO" gate="SHIELD" pin="D7"/>
 </segment>
 <segment>
@@
 <wire x1="78.74" y1="30.48" x2="81.28" y2="30.48" width="0.1524" layer="91"/>
 <label x="81.28" y="30.48" size="1.27" layer="95" xref="yes"/>
-<pinref part="ARDUINO" gate="G$1" pin="D8"/>
+<pinref part="ARDUINO" gate="SHIELD" pin="D8"/>
 </segment>
 <segment>
@@
 <wire x1="78.74" y1="27.94" x2="81.28" y2="27.94" width="0.1524" layer="91"/>
 <label x="81.28" y="27.94" size="1.27" layer="95" xref="yes"/>
-<pinref part="ARDUINO" gate="G$1" pin="*D9"/>
+<pinref part="ARDUINO" gate="SHIELD" pin="*D9"/>
 </segment>
 <segment>
@@
 <wire x1="78.74" y1="22.86" x2="81.28" y2="22.86" width="0.1524" layer="91"/>
 <label x="81.28" y="22.86" size="1.27" layer="95" xref="yes"/>
-<pinref part="ARDUINO" gate="G$1" pin="*D11"/>
+<pinref part="ARDUINO" gate="SHIELD" pin="*D11"/>
 </segment>
 </net>
@@
 <wire x1="78.74" y1="20.32" x2="81.28" y2="20.32" width="0.1524" layer="91"/>
 <label x="81.28" y="20.32" size="1.27" layer="95" xref="yes"/>
-<pinref part="ARDUINO" gate="G$1" pin="D12"/>
+<pinref part="ARDUINO" gate="SHIELD" pin="D12"/>
 </segment>
 </net>
@@
 <wire x1="78.74" y1="17.78" x2="81.28" y2="17.78" width="0.1524" layer="91"/>
 <label x="81.28" y="17.78" size="1.27" layer="95" xref="yes"/>
-<pinref part="ARDUINO" gate="G$1" pin="D13"/>
+<pinref part="ARDUINO" gate="SHIELD" pin="D13"/>
 </segment>
 </net>
@@
 <wire x1="53.34" y1="27.94" x2="33.02" y2="27.94" width="0.1524" layer="91"/>
 <pinref part="P+5" gate="G$1" pin="3.3V"/>
-<pinref part="ARDUINO" gate="G$1" pin="3.3V"/>
+<pinref part="ARDUINO" gate="SHIELD" pin="3.3V"/>
 </segment>
 <segment>
@@
 <wire x1="53.34" y1="33.02" x2="40.64" y2="33.02" width="0.1524" layer="91"/>
 <pinref part="P+6" gate="1" pin="V+"/>
-<pinref part="ARDUINO" gate="G$1" pin="VIN"/>
+<pinref part="ARDUINO" gate="SHIELD" pin="VIN"/>
 </segment>
 <segment>
@@
 <net name="GND" class="1">
 <segment>
-<pinref part="ARDUINO" gate="G$1" pin="GND@2"/>
-<pinref part="ARDUINO" gate="G$1" pin="GND@1"/>
+<pinref part="ARDUINO" gate="SHIELD" pin="GND@2"/>
+<pinref part="ARDUINO" gate="SHIELD" pin="GND@1"/>
 <wire x1="53.34" y1="22.86" x2="53.34" y2="20.32" width="0.1524" layer="91"/>
-<pinref part="ARDUINO" gate="G$1" pin="GND@0"/>
+<pinref part="ARDUINO" gate="SHIELD" pin="GND@0"/>
 <wire x1="53.34" y1="20.32" x2="53.34" y2="17.78" width="0.1524" layer="91"/>
 <junction x="53.34" y="20.32"/>
@@
 <net name="!RESET" class="0">
 <segment>
-<pinref part="ARDUINO" gate="G$1" pin="RES"/>
+<pinref part="ARDUINO" gate="SHIELD" pin="RES"/>
 <wire x1="53.34" y1="35.56" x2="43.18" y2="35.56" width="0.1524" layer="91"/>
 <label x="43.18" y="35.56" size="1.27" layer="95" rot="R90" xref="yes"/>
